File: src/power-thing.kicad_sch (KiCad schematic)
At the start: 4 parts, among them SW1 SW_DPST

Commit message: Adjustments
Parts:
- R1: value 1.5 MΩ ±10% -> 1.5±10% MΩ
Connections:
- net Black Wire: now also V1.1; no longer SW1.2, SW1.4, V1.2
- net at C1.1, R1.2, SW1.1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: now also V1.2; no longer V1.1
- new net Red Wire: SW1.2, SW1.4
Other:
- moved on the sheet: C1, R1, SW1, V1

Commit message: sync for bug tracking
Parts:
- removed V1: VSIN (EUROPLUG), symbol Simulation_SPICE:VSIN
- added P1: Conn_WallPlug_Earth, EVGA:IEC_320-C14_Panel_Mount, symbol Connector:Conn_WallPlug_Earth
- C1: footprint (none) -> EVGA:FTK_Capacitor
- R1: footprint (none) -> Resistor_THT:R_Axial_DIN0204_L3.6mm_D1.6mm_P5.08mm_Horizontal
- SW1: footprint (none) -> EVGA:EVGA_Switch
Connections:
- net at C1.1, R1.2, SW1.1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: now also P1.2 (AC_N)
- net Black Wire: no longer names the net of C1.2, R1.1
- net Black Wire: now also P1.1 (AC_P)
- net Red Wire: no longer names the net of SW1.2, SW1.4
- new net GNDPWR: P1.3 (EARTH)
Other:
- note added: "220~240 VAC 50Hz ADAM TECH - IEC-A-2"
- moved on the sheet: R1

Commit message: Ready For Review!
Connections:
- net GNDPWR is gone; now on net GND: P1.3 (EARTH)
- net at C1.1, P1.2 (AC_N), R1.2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: no longer SW1.3
- net at SW1.2: no longer SW1.4
Changed lines of the file:
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@@
+	)
+	(symbol
+		(lib_id "power:GND")
+		(at 86.36 158.75 180)
+		(unit 1)
+		(exclude_from_sim no)
+		(in_bom yes)
+		(on_board yes)
+		(dnp no)
+		(fields_autoplaced yes)
+		(property "Reference" "#PWR01"
+			(at 86.36 152.4 0)
+			(effects
+				(font
+					(size 1.27 1.27)
+				)
+				(hide yes)
+			)
+		)
+		(property "Value" "GND"
+			(at 86.36 153.67 0)
+			(effects
+				(font
+					(size 1.27 1.27)
+				)
+			)
+		)
+		(property "Footprint" ""
+			(at 86.36 158.75 0)
+			(effects
+				(font
+					(size 1.27 1.27)
+				)
+				(hide yes)
+			)
+		)
+		(property "Datasheet" ""
+			(at 86.36 158.75 0)
+			(effects
+				(font
+					(size 1.27 1.27)
+				)
+				(hide yes)
+			)
+		)
+		(property "Description" "Power symbol creates a global label with name \"GND\" , ground"
+			(at 86.36 158.75 0)
+			(effects
+				(font
+					(size 1.27 1.27)
+				)
+				(hide yes)
+			)
+		)
+		(pin "1"
+		)
+		(instances
+			(project "power-thing"
+				(path "/8766be43-8ceb-49b1-8438-758f0095b1c2"
+					(reference "#PWR01")
+					(unit 1)
+				)
+			)
+		)
 	)
 	(symbol
@@
 			)
 		)
-		(pin "3"
+		(pin "1"
 		)
 		(pin "2"
@@
 		(pin "1"
 		)
-		(pin "4"
+		(pin "2"
 		)
 		(instances
@@
 					(unit 1)
 				)
-			)
-		)
-	)
-	(symbol
-		(lib_id "power:GNDPWR")
-		(at 86.36 158.75 180)
-		(unit 1)
-		(exclude_from_sim no)
-		(in_bom yes)
-		(on_board yes)
-		(dnp no)
-		(fields_autoplaced yes)
-		(property "Reference" "#PWR01"
-			(at 86.36 153.67 0)
-			(effects
-				(font
-					(size 1.27 1.27)
-				)
-				(hide yes)
-			)
-		)
-		(property "Value" "GNDPWR"
-			(at 86.487 154.94 0)
-			(effects
-				(font
-					(size 1.27 1.27)
-				)
-			)
-		)
-		(property "Footprint" ""
-			(at 86.36 157.48 0)
-			(effects
-				(font
-					(size 1.27 1.27)
-				)
-				(hide yes)
-			)
-		)
-		(property "Datasheet" ""
-			(at 86.36 157.48 0)
-			(effects
-				(font
-					(size 1.27 1.27)
-				)
-				(hide yes)
-			)
-		)
-		(property "Description" "Power symbol creates a global label with name \"GNDPWR\" , global ground"
-			(at 86.36 158.75 0)
-			(effects
-				(font
-					(size 1.27 1.27)
-				)
-				(hide yes)
-			)
-		)
-		(pin "1"
-		)
-		(instances
-			(project "power-thing"
-				(path "/8766be43-8ceb-49b1-8438-758f0095b1c2"
-					(reference "#PWR01")
-					(unit 1)
-				)

Commit message: Review Adjustments
Parts:
- added J1, J2: 62409-1, 62409-1:TE_62409-1, symbol 62409-1:62409-1
Connections:
- net at C1.2, P1.1 (AC_P), R1.1: now also J1.1 (P1), J1.2 (P1)
- net at SW1.2: now also J2.1 (P1), J2.2 (P1)
