File: src/power-thing.kicad_pcb (KiCad board)
At the start: 2 copper layers, 32 x 46 mm, 4 parts, among them P1 Conn_WallPlug_Earth, SW1 SW_DPST

Commit message: Ready For Review!
Parts:
- added REF**: OSHW-Logo_7.5x8mm_Copper, Symbol:OSHW-Logo_7.5x8mm_Copper, B.Cu at (25.3, 27.3)
- moved R1 0.59 mm to (12.9, 9.09)
- moved P1 0.55 mm to (15.8, 19.3)
Connections:
- C1 pad 2: Net-(P1-AC_P) -> Net-(P1-AC_N)
Routing:
- net Net-(P1-AC_P): track 1.02 -> 0.00 mm
Other:
- outline, holes or cut-outs redrawn
- board text added: "OwO"

Commit message: Review Adjustments
Parts:
- removed the REF** at (25.3, 27.3)
- added J1: 62409-1, 62409-1:TE_62409-1, F.Cu at (3.30, 22.4)
- added J2: 62409-1, 62409-1:TE_62409-1, F.Cu at (3.17, 39.1)
- added REF**: OSHW-Logo_5.7x6mm_SilkScreen, Symbol:OSHW-Logo_5.7x6mm_SilkScreen, F.Cu at (23.7, 26.8)
Connections:
- C1 pad 1: Net-(P1-AC_P) -> Net-(P1-AC_N)
- C1 pad 2: Net-(P1-AC_N) -> Net-(P1-AC_P)
- P1 pad 1: Net-(P1-AC_P) -> Net-(P1-AC_N)
- P1 pad 2: Net-(P1-AC_N) -> Net-(P1-AC_P)
- R1 pad 1: Net-(P1-AC_P) -> Net-(P1-AC_N)
- R1 pad 2: Net-(P1-AC_N) -> Net-(P1-AC_P)
Routing:
- net Net-(P1-AC_P): vias 1 -> 0
- net Net-(J2-P1-Pad1): vias 1 -> 0
Other:
- outline, holes or cut-outs redrawn

Commit message: Pre-Release
Parts:
- moved J1 1.50 mm to (1.80, 22.5)
Other:
- board text added: "BLACK"
- board text added: "RED"
Changed lines of the file:
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@@
 			(solder_mask_margin 0.102)
 		)
-		(model "/home/kreyren/Downloads/stuffson/62409-1.step"
+		(model "${KIPRJMOD}/62409-1.pretty/62409-1.step"
 			(offset
 				(xyz 0 0 0)
@@
 			(pintype "passive")
 		)
-		(model "${KICAD8_3DMODEL_DIR}/Resistor_THT.3dshapes/R_Axial_DIN0204_L3.6mm_D1.6mm_P5.08mm_Horizontal.wrl"
-			(hide yes)
+		(model "${KICAD8_3DMODEL_DIR}/Resistor_THT.3dshapes/R_Axial_DIN0207_L6.3mm_D2.5mm_P10.16mm_Horizontal.wrl"
 			(offset
-				(xyz 0 0 0)
+				(xyz -3 0 0)
 			)
 			(scale
-				(xyz 1 1 1)
+				(xyz 1.075 0.9 0.8)
 			)
 			(rotate
@@
 		(at 15.5 4.5)
 		(property "Reference" "C1"
-			(at -3.8 1.5 0)
+			(at -5.205868 -1.325518 0)
 			(unlocked yes)
 			(layer "F.SilkS")
@@
 			(fill none)
 			(layer "F.SilkS")
+		)
+		(fp_text user "+340VAC 0.33uF"
+			(at -5.5 2.368968 0)
+			(unlocked yes)
+			(layer "F.SilkS")
+			(effects
+				(font
+					(size 1.25 1.25)
+					(thickness 0.2)
+				)
+				(justify left bottom)
+			)
 		)
 		(fp_text user "${REFERENCE}"
@@
 			(net 2 "Net-(P1-AC_P)")
 			(pintype "passive")
+		)
+		(model "/home/kreyren/Downloads/MKP4G033305B00MSSD.STEP"
+			(offset
+				(xyz 0 0 -1.5)
+			)
+			(scale
+				(xyz 1 1 1)
+			)
+			(rotate
+				(xyz 90 0 0)
+			)
 		)
 	)
@@
 			(pintype "power_out")
 		)
+		(model "${KIPRJMOD}/power-socket-c14-1.pretty/powerSocket.stp"
+			(offset
+				(xyz 0.5 -0.5 -2.5)
+			)
+			(scale
+				(xyz 1 1 1)
+			)
+			(rotate
+				(xyz 0 -180 180)
+			)
+		)
 	)
 	(footprint "EVGA:EVGA_Switch"
@@
 			(pintype "passive")
 		)
+		(model "${KIPRJMOD}/R1973BBLKGILFF1/R1973BBLKGILFF1--3DModel-STEP-520916.STEP"
+			(offset
+				(xyz 1 0 -3)
+			)
+			(scale
+				(xyz 1 1 1)
+			)
+			(rotate
+				(xyz -180 0 0)
+			)
+		)
 	)
 	(footprint "62409-1:TE_62409-1"
 		(layer "F.Cu")
-		(at 3.302 22.352 90)
+		(at 1.801183 22.458719 90)
 		(property "Reference" "J1"
-			(at 0 0 270)
+			(at 0 0 -90)
 			(layer "F.SilkS")
 			(effects
@@
 			(solder_mask_margin 0.102)
 		)
-		(model "/home/kreyren/Downloads/stuffson/62409-1.step"
+		(model "${KIPRJMOD}/62409-1.pretty/62409-1.step"
 			(offset
 				(xyz 0 0 0)
@@
 	(gr_rect
 		(start 0.3 0.3)
-		(end 13.8 5.35)
+		(end 12.3 5.35)
 		(stroke
 			(width 0)
@@
 	(gr_poly
 		(pts
-			(xy 13.75 16.575) (xy 7.75 16.575) (xy 10.45 20.25)
+			(xy 12.3 16.55) (xy 7.75 16.575) (xy 10.606836 19.79019)
 		)
 		(stroke
@@
 	(gr_poly
 		(pts
-			(xy 17.16 16.38) (xy 21.425 20.4) (xy 23.75 16.38)
+			(xy 18.66 16.38) (xy 21.425 20.4) (xy 23.75 16.38)
 		)
 		(stroke
@@
 		(fill solid)
 		(layer "F.Cu")
-		(net 1)
+		(net 2)
 	)
 	(gr_rect
 		(start 7.8 5.35)
-		(end 13.8 16.55)
+		(end 12.3 16.55)
 		(stroke
 			(width 0)
@@
 	)
 	(gr_rect
-		(start 25.675 5.4)
-		(end 31.7 45.7)
+		(start 25.675 5.5)
+		(end 31.7 45.3)
 		(stroke
 			(width 0)
@@
 	)
 	(gr_rect
-		(start 17.16 0.3)
+		(start 18.66 0.3)
 		(end 31.7 5.4)
 		(stroke
@@
 		(fill solid)
 		(layer "F.Cu")
-		(net 1)
+		(net 2)
 	)
 	(gr_circle
@@
 	)
 	(gr_rect
-		(start 17.16 5.4)
+		(start 18.66 5.4)
 		(end 23.75 16.38)
 		(stroke
@@
 		(fill solid)
 		(layer "F.Cu")
-		(net 1)
+		(net 2)
 	)
 	(gr_poly
@@
 		(fill solid)
 		(layer "B.Cu")
-		(net 1)
+		(net 2)
 	)
 	(gr_poly
@@
 		(fill solid)
 		(layer "B.Cu")
-		(net 1)
+		(net 2)
 	)
 	(gr_circle
@@
 		(fill solid)
 		(layer "B.Cu")
-		(net 1)
+		(net 2)
 	)
 	(gr_circle
@@
 		(fill solid)
 		(layer "B.Cu")
-		(net 1)
+		(net 2)
 	)
 	(gr_circle
@@
 		(fill solid)
 		(layer "B.Cu")
-		(net 1)
+		(net 2)
 	)
 	(gr_circle
@@
 		(fill solid)
 		(layer "B.Cu")
-		(net 1)
+		(net 2)
 	)
 	(gr_circle
@@
 		(fill solid)
 		(layer "B.Cu")
-		(net 1)
+		(net 2)
 	)
 	(gr_circle
@@
 		(fill solid)
 		(layer "B.Cu")
-		(net 1)
+		(net 2)
 	)
 	(gr_circle
@@
 		(fill solid)
 		(layer "B.Cu")
-		(net 1)
+		(net 2)
 	)
 	(gr_circle
@@
 		(fill solid)
 		(layer "B.Cu")
-		(net 1)
+		(net 2)
 	)
 	(gr_circle
@@
 		(fill solid)
 		(layer "B.Cu")
-		(net 1)
+		(net 2)
 	)
 	(gr_arc
@@
 			)
 			(justify left bottom)
+		)
+	)
+	(gr_text "BLACK"
+		(at 4.304655 24.512474 90)
+		(layer "F.SilkS")
+		(effects
+			(font
+				(size 1 1)
+				(thickness 0.1)
+			)
+			(justify left bottom)
+		)
+	)
+	(gr_text "RED"
+		(at 5.96935 40.551697 90)
+		(layer "F.SilkS")
+		(effects
+			(font
+				(size 1 1)
+				(thickness 0.1)
+			)
+			(justify left bottom)
