File: src/evga1000g2db.kicad_pcb (KiCad board)
At the start: 2 copper layers, 32 x 46 mm, 12 parts, among them J1 62409-1, J2 62409-1, P1 Conn_WallPlug_Earth, SW1 SW_DPST

Commit message: More adjustments
Parts:
- moved REF** 0.79 mm to (56.8, 118.8)
Changed lines of the file:
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@@
 			(drillshape 0)
 			(scaleselection 1)
-			(outputdirectory "../build/")
+			(outputdirectory "../build/drill_files")
 		)
 	)
@@
 	(footprint "Symbol:KiCad-Logo2_20mm_SilkScreen"
 		(layer "F.Cu")
-		(at 57 118)
+		(at 56.75 118.75)
 		(descr "KiCad Logo")
 		(tags "Logo KiCad")
@@
 	(dimension
 		(type aligned)
-		(layer "F.SilkS")
+		(layer "Cmts.User")
 		(pts
-			(xy 33.641969 29.820249) (xy 65.641969 29.820249)
+			(xy 33.641969 29.820249) (xy 33.641969 75.820249)
 		)
-		(height -4.5)
-		(gr_text "32.0000 mm"
-			(at 49.641969 24.220249 0)
-			(layer "F.SilkS")
+		(height 7.141968)
+		(gr_text "46.0000 mm"
+			(at 25.350001 52.820249 90)
+			(layer "Cmts.User")
 			(effects
 				(font
 					(size 1 1)
-					(thickness 0.1)
+					(thickness 0.15)
 				)
 			)
@@
 	(dimension
 		(type aligned)
-		(layer "F.SilkS")
+		(layer "Cmts.User")
 		(pts
-			(xy 33.641969 29.820249) (xy 33.641969 75.820249)
+			(xy 65.641969 29.820249) (xy 33.641969 29.820249)
 		)
-		(height 5.942274)
-		(gr_text "46.0000 mm"
-			(at 26.599695 52.820249 90)
-			(layer "F.SilkS")
+		(height 6.570248)
+		(gr_text "32.0000 mm"
+			(at 49.641969 22.100001 0)
+			(layer "Cmts.User")
 			(effects
 				(font
 					(size 1 1)
-					(thickness 0.1)
+					(thickness 0.15)
 				)
 			)

Commit message: sync
Parts:
- moved REF** 105.2 mm to (143.1, 178.8)
- moved REF** 1.38 mm to (37.5, 45.6)
- moved J1 0.63 mm to (35.7, 51.7)
Other:
- board text added: "FABRICATING NOTES"
- board text added: "RoHS"
- board text removed: "Requires >=2 oz copper"
